Commit message: rviz config update

File: urdf/zortax.urdf (robot description, URDF)
Before this commit: robot myrobot, 0 links, 0 joints
Links:
- added link base_link; visual mesh filename=package://zortax_robotic_arm/meshes/part1.dae
- added link part2; visual mesh filename=package://zortax_robotic_arm/meshes/part2.dae
- added link part3; visual mesh filename=package://zortax_robotic_arm/meshes/part3.dae
Joints:
- added joint base_to_part1: type continuous, parent base_link, child part2, origin xyz=0 0 100, axis 0 1 0
- added joint part2_to_part3: type continuous, parent part2, child part3, axis 0 1 0
