Commit message: dkin done

File: urdf/simple.urdf (robot description, URDF)
Before this commit: robot myrobot, 5 links, 4 joints
Links:
- link base_link: geometry visual box size=0.1 0.1 0.12
- link part1: geometry visual box size=0.05 0.05 0.0805
- link part2: geometry visual cylinder length=0.1575 radius=0.030
- link part3: geometry visual cylinder length=0.18334 radius=0.025
- link part4: geometry visual cylinder length=0.14616 radius=0.015
Joints:
- joint joint0: origin xyz=0 0 1.2 rpy=0 0 0 -> xyz=0 0 0.12 rpy=0 0 0
- joint joint1: origin xyz=0 0 0.85 rpy=0 0 0 -> xyz=0 0 0.0805 rpy=0 0 0
- joint joint2: origin xyz=0 0 1.575 rpy=0 0 0 -> xyz=0 0 0.1575 rpy=0 1.57 0
- joint joint3: origin xyz=0 0 1.8334 rpy=0 0 0 -> xyz=0 0 0.18334 rpy=0 0.785 0; type continuous -> fixed
